File: PCB/477.sch (EAGLE design)
At the start: 48 parts, among them IC2 STM32F407VGT6, U2 ESP8266-12E/ESP-12E, Y1 8MHz

Commit message: Updated PCB files
Modified main PCB and added the second PCB for relay
Parts:
- removed PD, PE, PE1: (no value), SparkFun-Connectors:CONN_06NO_SILK_FEMALE_PTH
- added ADC, NRST: (no value), SparkFun-Connectors:CONN_01
- added LED, STL: (no value), SparkFun-Connectors:CONN_03
- added P/S: (no value), SparkFun-Connectors:CONN_07
- added R1, R2, R3: 150, SparkFun-Resistors:150OHM-0603-1/10W-1%
- added TEST: (no value), SparkFun-Connectors:CONN_04
- renumbered PA to MISC, PC to BTN
Connections:
- net PA2 renamed TX2
- net PA3 renamed RX2
- net PC10 renamed B/STP
- net PC11 renamed B/RSTA
- removed net PA0: IC2.PA0, MISC.5
- removed net PA5: IC2.PA5, MISC.4
- removed net PB2: IC2.PB2, PE1.4, R5.1, R6.1
- removed net PB6: IC2.PB6, PE1.2
- removed net PB7: IC2.PB7, PE1.1
- removed net PD1: IC2.PD1, PD.1
- removed net PD2: IC2.PD2, PD.2
- removed net PD3: IC2.PD3, PD.3
- removed net PD4: IC2.PD4, PD.4
- removed net PD5: IC2.PD5, PD.5
- removed net PD6: IC2.PD6, PD.6
- removed net PE2: IC2.PE2, PE.2
- removed net PE3: IC2.PE3, PE.3
- removed net PE4: IC2.PE4, PE.4
- removed net PE5: IC2.PE5, PE.5
- removed net PE6: IC2.PE6, PE.6
- new net ADC: ADC.1, IC2.PA0
- new net BOOT1: IC2.PB2, R5.1, R6.1
- new net L/ERR: LED.2, R2.1
- new net L/PWR: LED.3, R3.1
- new net L/WRK: LED.1, R1.1
- new net N$1: IC2.PA4, R3.2
- new net N$2: IC2.PA5, R2.2
- new net N$4: IC2.PA6, R1.2
- new net P/PUMP: IC2.PD1, P/S.2
- new net P/RLY: IC2.PD0, P/S.1
- new net PA7: IC2.PA7, TEST.4
- new net PC12: IC2.PC12, TEST.1
- new net RX3: IC2.PB11, MISC.1
- new net SCL: IC2.PB6, MISC.4
- new net SDA: IC2.PB7, MISC.3
- new net SOL1: IC2.PD2, P/S.3
- new net SOL2: IC2.PD3, P/S.4
- new net SOL3: IC2.PD4, P/S.5
- new net SOL4: IC2.PD5, P/S.6
- new net SOLAIR: IC2.PD6, P/S.7
- new net TX3: IC2.PB10, MISC.2
- net EN: now also MISC.5; no longer MISC.3
- net GND: no longer PE.1
- net NRST: now also NRST.1
- net PA13: now also STL.3; no longer MISC.2
- net PA14: now also STL.2; no longer MISC.1
- net PB0: now also TEST.3; no longer PE1.6
- net PB1: now also TEST.2; no longer PE1.5
- net PB3: now also STL.1; no longer PE1.3
Other:
- moved on the sheet: C1, C2, JP1, JP2, R5, R6, R7, R8
